File: Schematics/SDRrecV6/Complete Schematic V6.kicad_sch (KiCad schematic)
At the start: 58 parts, among them J1 Conn_Coaxial, J2 SJ1-3525N, U1 Si5351A-B-GT, U2 SN74CBT3253, U3 LT6231, Y1 Crystal_GND24_Small

Commit message: updates
Parts:
- J2: footprint (none) -> CUI_SJ1-3225N:CUI_SJ1-3525N
Changed lines of the file:
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@@
       (effects (font (size 1.27 1.27)) (justify right))
     )
-    (property "Footprint" "" (id 2) (at 313.69 85.09 0)
+    (property "Footprint" "CUI_SJ1-3225N:CUI_SJ1-3525N" (id 2) (at 313.69 85.09 0)
       (effects (font (size 1.27 1.27)) (justify left bottom) hide)
     )
